File: NeoPixel-addressable/Arduino_WS_Led_Controller/Arduino_WS_Led_Controller.kicad_pcb (KiCad board)
At the start: 2 copper layers, 19 parts, among them J1 Terminal to WS2815 12V Strips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, J2 Terminal to MAX4466, J3 Terminal PWR, U1 WeMos_D1_mini, U2 LM2674N-3.3/NOPB, U3 TXB0104D, U4 LM317_TO-220

Commit message: Updates
Parts:
- moved R2 7.62 mm to (259.1, 163.8), turned to 180 degrees
- moved D2 2.54 mm to (247.7, 176.5), turned to 180 degrees
- moved U3 1.80 mm to (221.0, 139.7)
- moved R4 1.27 mm to (237.5, 135.9)
Routing:
- net 12VDC: track 0.00 -> 170.2 mm
- net GND: track 0.00 -> 59.6 mm
- net Net-(C3-Pad1): track 0.00 -> 20.5 mm
- net Net-(D2-Pad2): track 0.00 -> 10.7 mm
- added copper zone on B.Cu, net GND
- added copper zone on F.Cu, net GND
Other:
- board text added: "12V"
- board text added: "5V"
- board text added: "Dout"
- board text added: "From Power"
- board text added: "GND"
- board text added: "MIC"
- board text added: "To Led Strip"
- board text added: "To MAX4466"

Commit message: Getting the PCB set
Parts:
- added U5: MOUNTINGHOLE3.0THIN, MountingHole:MountingHole_3.2mm_M3, F.Cu at (196.2, 64.8)
- added U6: MOUNTINGHOLE3.0THIN, MountingHole:MountingHole_3.2mm_M3, F.Cu at (196.2, 125.7)
- added U7: MOUNTINGHOLE3.0THIN, MountingHole:MountingHole_3.2mm_M3, F.Cu at (128.9, 64.8)
- added U8: MOUNTINGHOLE3.0THIN, MountingHole:MountingHole_3.2mm_M3, F.Cu at (128.9, 125.7)
- U3: moved to B.Cu
- moved R3 114.9 mm to (137.2, 77.5), turned to 270 degrees
- moved J2 112.4 mm to (186.7, 82.5)
- moved R4 108.0 mm to (142.2, 85.1), turned to 90 degrees
- moved R2 104.1 mm to (176.5, 100.3)
- moved J1 102.9 mm to (186.7, 118.1)
- moved L1 102.9 mm to (162.6, 87.6)
- moved C2 102.8 mm to (172.7, 109.9), turned to 270 degrees
- moved C5 102.7 mm to (150.5, 72.4)
- moved C3 102.2 mm to (171.4, 73.7)
- moved U2 102.2 mm to (176.5, 82.5)
- moved C1 102.2 mm to (165.1, 72.4)
- moved C4 102.2 mm to (162.6, 78.7)
- moved D1 102.2 mm to (168.9, 96.5)
- moved R1 102.2 mm to (162.6, 108.0)
- moved U1 102.2 mm to (133.3, 96.5)
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Routing:
- net 12VDC: track 170.2 -> 0.00 mm
- net 5VDC: track 0.00 -> 137.3 mm
- net 3V3DC: track 0.00 -> 83.0 mm
- net Net-(J2-Pad2): track 0.00 -> 71.2 mm
- net GND: track 59.6 -> 0.00 mm
- net Net-(R2-Pad2): track 0.00 -> 46.4 mm
- net Net-(U1-Pad2): track 0.00 -> 19.1 mm
- net Net-(C3-Pad1): track 20.5 -> 39.4 mm
- net Net-(J1-Pad3): track 0.00 -> 13.4 mm
- net Net-(U1-Pad7): track 0.00 -> 10.1 mm
- net Net-(C3-Pad2): track 0.00 -> 8.92 mm
- net Net-(R3-Pad1): track 0.00 -> 5.08 mm
- net Net-(D2-Pad2): track 10.7 -> 10.2 mm
- added copper zone on F.Cu, net 12VDC
- removed copper zone on F.Cu, net GND
Other:
- board outline added: 74.9 x 68.6 mm
- board text added: "WS2815 LED CONTROLLER v0.5 Randall Shutt Randall@randallman.net"
