File: NeoPixel-addressable/Arduino_WS_Led_Controller/Arduino_WS_Led_Controller.kicad_pcb (KiCad board)
At the start: 2 copper layers, 74.9 x 68.6 mm, 23 parts, among them J1 Terminal to WS2815 12V Strips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, J2 Terminal to MAX4466, J3 Terminal PWR, U1 WeMos_D1_mini, U2 LM2674N-3.3/NOPB, U3 TXB0104D, U4 LM317_TO-220, U5 MOUNTINGHOLE3.0THIN, U6 MOUNTINGHOLE3.0THIN, U7 MOUNTINGHOLE3.0THIN, U8 MOUNTINGHOLE3.0THIN

Commit message: Interim commit
Parts:
- C5: footprint Capacitor_THT:C_Disc_D3.0mm_W2.0mm_P2.50mm -> Capacitor_THT:C_Disc_D7.5mm_W5.0mm_P5.00mm
- moved R4 3.81 mm to (142.2, 81.3), turned to 0 degrees
- moved C5 1.42 mm to (151.1, 73.7)
Connections:
- R4 pad 1: GND -> Net-(R3-Pad1)
Routing:
- net 5VDC: track 138.4 -> 155.1 mm
- net Net-(R3-Pad1): track 5.08 -> 11.7 mm
Other:
- board text added: "WS2815 LED CONTROLLER v0.6 Randall Shutt Randall@randallman.net"
- board text removed: "WS2815 LED CONTROLLER v0.5 Randall Shutt Randall@randallman.net"
