File: NeoPixel-addressable/Arduino_WS_Led_Controller/Arduino_WS_Led_Controller.sch (KiCad schematic (older format))
At the start: 19 parts, among them J1 Terminal to WS2815 12V Strips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, J2 Terminal to MAX4466, J3 Terminal PWR, U1 WeMos_D1_mini, U2 LM2674N-3.3/NOPB, U3 TXB0104D, U4 LM317_TO-220

Commit message: Getting the PCB set
Parts:
- added U5, U6, U7, U8: MOUNTINGHOLE3.0THIN, MountingHole:MountingHole_3.2mm_M3, symbol Arduino_WS_Led_Controller-eagle-import:MOUNTINGHOLE3.0THIN
Other:
- moved on the sheet: C5, R3, R4, U4
Changed lines of the file:
@@
 L Regulator_Linear:LM317_TO-220 U4
 U 1 1 616E6268
-P 6100 2250
-F 0 "U4" H 6100 2492 50  0000 C CNN
-F 1 "LM317_TO-220" H 6100 2401 50  0000 C CNN
-F 2 "Package_TO_SOT_THT:TO-220-3_Vertical" H 6100 2500 50  0001 C CIN
-F 3 "http://www.ti.com/lit/ds/symlink/lm317.pdf" H 6100 2250 50  0001 C CNN
-	1    6100 2250
-	1    0    0    -1
-$EndComp
-Text GLabel 5500 2250 0    50   Input ~ 0
+P 6000 2350
+F 0 "U4" H 6000 2592 50  0000 C CNN
+F 1 "LM317_TO-220" H 6000 2501 50  0000 C CNN
+F 2 "Package_TO_SOT_THT:TO-220-3_Vertical" H 6000 2600 50  0001 C CIN
+F 3 "http://www.ti.com/lit/ds/symlink/lm317.pdf" H 6000 2350 50  0001 C CNN
+	1    6000 2350
+	1    0    0    -1
+$EndComp
+Text GLabel 5400 2350 0    50   Input ~ 0
 12VDC
-Text GLabel 6850 2250 2    50   Output ~ 0
+Text GLabel 6750 2350 2    50   Output ~ 0
 5VDC
 $Comp
 L Device:R R4
 U 1 1 616E75C2
-P 6650 2500
-F 0 "R4" H 6580 2454 50  0000 R CNN
-F 1 "330" H 6580 2545 50  0000 R CNN
-F 2 "Resistor_THT:R_Axial_DIN0207_L6.3mm_D2.5mm_P7.62mm_Horizontal" V 6580 2500 50  0001 C CNN
-F 3 "~" H 6650 2500 50  0001 C CNN
-	1    6650 2500
+P 6550 2600
+F 0 "R4" H 6480 2554 50  0000 R CNN
+F 1 "330" H 6480 2645 50  0000 R CNN
+F 2 "Resistor_THT:R_Axial_DIN0207_L6.3mm_D2.5mm_P7.62mm_Horizontal" V 6480 2600 50  0001 C CNN
+F 3 "~" H 6550 2600 50  0001 C CNN
+	1    6550 2600
 	-1   0    0    1
 $EndComp
 Wire Wire Line
-	6400 2250 6650 2250
-Wire Wire Line
-	6650 2350 6650 2250
-Connection ~ 6650 2250
-Wire Wire Line
-	6650 2250 6850 2250
-Wire Wire Line
-	6650 2650 6650 2800
+	6300 2350 6550 2350
+Wire Wire Line
+	6550 2450 6550 2350
+Connection ~ 6550 2350
+Wire Wire Line
+	6550 2350 6750 2350
+Wire Wire Line
+	6550 2750 6550 2900
 $Comp
 L Device:R R3
 U 1 1 616EACA8
-P 6350 2800
-F 0 "R3" V 6557 2800 50  0000 C CNN
-F 1 "1000" V 6466 2800 50  0000 C CNN
-F 2 "Resistor_THT:R_Axial_DIN0207_L6.3mm_D2.5mm_P7.62mm_Horizontal" V 6280 2800 50  0001 C CNN
-F 3 "~" H 6350 2800 50  0001 C CNN
-	1    6350 2800
+P 6250 2900
+F 0 "R3" V 6457 2900 50  0000 C CNN
+F 1 "1000" V 6366 2900 50  0000 C CNN
+F 2 "Resistor_THT:R_Axial_DIN0207_L6.3mm_D2.5mm_P7.62mm_Horizontal" V 6180 2900 50  0001 C CNN
+F 3 "~" H 6250 2900 50  0001 C CNN
+	1    6250 2900
 	0    -1   -1   0
 $EndComp
 Wire Wire Line
-	6100 2550 6100 2800
-Wire Wire Line
-	6100 2800 6200 2800
-Wire Wire Line
-	6500 2800 6650 2800
-Connection ~ 6650 2800
-Wire Wire Line
-	6650 2800 6650 2950
+	6000 2650 6000 2900
+Wire Wire Line
+	6000 2900 6100 2900
+Wire Wire Line
+	6400 2900 6550 2900
+Connection ~ 6550 2900
+Wire Wire Line
+	6550 2900 6550 3050
 $Comp
 L power:+5V #PWR07
@@
 L power:GND #PWR010
 U 1 1 6174D4B3
-P 6100 3050
-F 0 "#PWR010" H 6100 2800 50  0001 C CNN
-F 1 "GND" H 6100 2900 50  0000 C CNN
-F 2 "" H 6100 3050 50  0001 C CNN
-F 3 "" H 6100 3050 50  0001 C CNN
-	1    6100 3050
+P 6000 3150
+F 0 "#PWR010" H 6000 2900 50  0001 C CNN
+F 1 "GND" H 6000 3000 50  0000 C CNN
+F 2 "" H 6000 3150 50  0001 C CNN
+F 3 "" H 6000 3150 50  0001 C CNN
+	1    6000 3150
 	1    0    0    -1
 $EndComp
@@
 Connection ~ 6100 1350
 Wire Wire Line
-	5800 2250 5650 2250
+	5700 2350 5550 2350
 $Comp
 L Device:C C5
 U 1 1 617A57C0
-P 5650 2500
-F 0 "C5" H 5765 2546 50  0000 L CNN
-F 1 "0.1uF" H 5765 2455 50  0000 L CNN
-F 2 "Capacitor_THT:C_Disc_D3.0mm_W2.0mm_P2.50mm" H 5688 2350 50  0001 C CNN
-F 3 "~" H 5650 2500 50  0001 C CNN
-	1    5650 2500
-	1    0    0    -1
-$EndComp
-Wire Wire Line
-	5650 2350 5650 2250
-Connection ~ 5650 2250
-Wire Wire Line
-	5650 2250 5500 2250
-Wire Wire Line
-	5650 2950 6100 2950
-Wire Wire Line
-	5650 2650 5650 2950
-Wire Wire Line
-	6100 3050 6100 2950
-Connection ~ 6100 2950
-Wire Wire Line
-	6100 2950 6650 2950
+P 5550 2600
+F 0 "C5" H 5665 2646 50  0000 L CNN
+F 1 "0.1uF" H 5665 2555 50  0000 L CNN
+F 2 "Capacitor_THT:C_Disc_D3.0mm_W2.0mm_P2.50mm" H 5588 2450 50  0001 C CNN
+F 3 "~" H 5550 2600 50  0001 C CNN
+	1    5550 2600
+	1    0    0    -1
+$EndComp
+Wire Wire Line
+	5550 2450 5550 2350
+Connection ~ 5550 2350
+Wire Wire Line
+	5550 2350 5400 2350
+Wire Wire Line
+	5550 3050 6000 3050
+Wire Wire Line
+	5550 2750 5550 3050
+Wire Wire Line
+	6000 3150 6000 3050
+Connection ~ 6000 3050
+Wire Wire Line
+	6000 3050 6550 3050
 Wire Wire Line
 	2850 4100 2550 4100
@@
 Wire Wire Line
 	3050 4050 3050 4100
+$Comp
+L Arduino_WS_Led_Controller-eagle-import:MOUNTINGHOLE3.0THIN U7
+U 1 1 61816C7E
+P 950 200
+F 0 "U7" H 1000 250 50  0001 C CNN
+F 1 "MOUNTINGHOLE3.0THIN" H 950 200 50  0001 C CNN
+F 2 "MountingHole:MountingHole_3.2mm_M3" H 950 200 50  0001 C CNN
+F 3 "" H 950 200 50  0001 C CNN
+	1    950  200
+	1    0    0    -1
+$EndComp
+$Comp
+L Arduino_WS_Led_Controller-eagle-import:MOUNTINGHOLE3.0THIN U5
+U 1 1 61821DC1
+P 200 200
+F 0 "U5" H 250 250 50  0001 C CNN
+F 1 "MOUNTINGHOLE3.0THIN" H 200 200 50  0001 C CNN
+F 2 "MountingHole:MountingHole_3.2mm_M3" H 200 200 50  0001 C CNN
+F 3 "" H 200 200 50  0001 C CNN
+	1    200  200
+	1    0    0    -1
+$EndComp
+$Comp
+L Arduino_WS_Led_Controller-eagle-import:MOUNTINGHOLE3.0THIN U6
+U 1 1 61823D4B
+P 450 200
+F 0 "U6" H 500 250 50  0001 C CNN
+F 1 "MOUNTINGHOLE3.0THIN" H 450 200 50  0001 C CNN
+F 2 "MountingHole:MountingHole_3.2mm_M3" H 450 200 50  0001 C CNN
+F 3 "" H 450 200 50  0001 C CNN
+	1    450  200
+	1    0    0    -1
+$EndComp
+$Comp
+L Arduino_WS_Led_Controller-eagle-import:MOUNTINGHOLE3.0THIN U8
+U 1 1 61827D6A
+P 700 200
+F 0 "U8" H 750 250 50  0001 C CNN
+F 1 "MOUNTINGHOLE3.0THIN" H 700 200 50  0001 C CNN
+F 2 "MountingHole:MountingHole_3.2mm_M3" H 700 200 50  0001 C CNN
+F 3 "" H 700 200 50  0001 C CNN
+	1    700  200
+	1    0    0    -1
+$EndComp
 $EndSCHEMATC
