File: NeoPixel-addressable/Arduino_WS_Led_Controller/Arduino_WS_Led_Controller_Oops_Working.sch (KiCad schematic (older format))
At the start: 23 parts, among them J1 Terminal to WS2815 12V Strips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, J2 Terminal to MAX4466, J3 Terminal PWR, U1 WeMos_D1_mini, U2 LM2674N-3.3/NOPB, U3 TXB0104D, U4 LM317_TO-220, U5 MOUNTINGHOLE3.0THIN, U6 MOUNTINGHOLE3.0THIN, U7 MOUNTINGHOLE3.0THIN, U8 MOUNTINGHOLE3.0THIN

Commit message: Interim commit
Parts:
- C1, C4: footprint Capacitor_THT:CP_Radial_D5.0mm_P2.00mm -> Capacitor_THT:CP_Radial_D8.0mm_P3.50mm
- C3, C5: footprint Capacitor_THT:C_Disc_D7.5mm_W5.0mm_P5.00mm -> Capacitor_THT:C_Disc_D5.0mm_W2.5mm_P5.00mm
- D2: footprint LED_THT:LED_D3.0mm_Clear -> LED_THT:LED_D5.0mm_Clear
Changed lines of the file:
@@
 F 0 "D2" H 4000 2200 50  0000 R CNN
 F 1 "LED" H 3850 2200 50  0000 R CNN
-F 2 "LED_THT:LED_D3.0mm_Clear" H 4000 2550 50  0001 C CNN
+F 2 "LED_THT:LED_D5.0mm_Clear" H 4000 2550 50  0001 C CNN
 F 3 "~" H 3900 2350 50  0001 C CNN
 	1    3900 2350
@@
 F 0 "C1" H 1918 1146 50  0000 L CNN
 F 1 "100uF OSCON-SEP" H 1550 950 50  0000 L CNN
-F 2 "Capacitor_THT:CP_Radial_D5.0mm_P2.00mm" H 1838 950 50  0001 C CNN
+F 2 "Capacitor_THT:CP_Radial_D8.0mm_P3.50mm" H 1838 950 50  0001 C CNN
 F 3 "~" H 1800 1100 50  0001 C CNN
 	1    1800 1100
@@
 F 0 "C3" V 3248 1150 50  0000 C CNN
 F 1 "0.01uF" V 3339 1150 50  0000 C CNN
-F 2 "Capacitor_THT:C_Disc_D7.5mm_W5.0mm_P5.00mm" H 3538 1000 50  0001 C CNN
+F 2 "Capacitor_THT:C_Disc_D5.0mm_W2.5mm_P5.00mm" H 3538 1000 50  0001 C CNN
 F 3 "~" H 3500 1150 50  0001 C CNN
 	1    3500 1150
@@
 F 0 "C4" H 4568 1546 50  0000 L CNN
 F 1 "100uF OSCON-SEP" H 4200 1400 50  0000 L CNN
-F 2 "Capacitor_THT:CP_Radial_D5.0mm_P2.00mm" H 4488 1350 50  0001 C CNN
+F 2 "Capacitor_THT:CP_Radial_D8.0mm_P3.50mm" H 4488 1350 50  0001 C CNN
 F 3 "~" H 4450 1500 50  0001 C CNN
 	1    4450 1500
@@
 F 0 "C5" H 5665 2646 50  0000 L CNN
 F 1 "0.1uF" H 5665 2555 50  0000 L CNN
-F 2 "Capacitor_THT:C_Disc_D7.5mm_W5.0mm_P5.00mm" H 5588 2450 50  0001 C CNN
+F 2 "Capacitor_THT:C_Disc_D5.0mm_W2.5mm_P5.00mm" H 5588 2450 50  0001 C CNN
 F 3 "~" H 5550 2600 50  0001 C CNN
 	1    5550 2600
